Commit message: Updated urdf to have L1L2 joint fixed and set range correctly if someone chooses to model the joint as a resolute joint.

File: ezgripper_driver/urdf/ezgripper_dual_IM.urdf.xacro (robot description, xacro)
@@ -161,5 +161,5 @@
       <origin xyz="0.052 0 0" rpy="0 0 0"/>
       <axis xyz="0 1 0"/>
-      <limit lower="-.27" upper="1.57075" effort="1" velocity="3.67"/>
+      <limit lower="0.0" upper="1.7" effort="1" velocity="3.67"/>
       <xacro:if value="${mimic_test}">
            <mimic joint="${prefix}_ezgripper_knuckle_L1_L2_1"/>
