Commit message: Fixed triple gripper URDF - need to upgrade to Gazebo 9

File: ezgripper_description/urdf/ezgripper_single_mount.urdf.xacro (robot description, xacro)
@@ -183,5 +183,5 @@
     <!-- transmissions for Gazebo -->
 <xacro:macro name="ezgripper_knuckle_trans" params="prefix postfix">
-   <transmission name="${prefix}_ezgripper_trans_${postfix}">
+   <transmission name="${prefix}_ezgripper_knuckle_${postfix}">
       <type>transmission_interface/SimpleTransmission</type>
       <joint name="${prefix}_ezgripper_knuckle_palm_L1_${postfix}">

File: ezgripper_description/urdf/ezgripper_triple_mount.urdf.xacro (robot description, xacro)
@@ -193,5 +193,5 @@
    <transmission name="${prefix}_ezgripper_trans_${postfix}">
       <type>transmission_interface/SimpleTransmission</type>
-      <joint name="${prefix}_ezgripper_knuckle_${postfix}">
+      <joint name="${prefix}_ezgripper_knuckle_palm_L1_${postfix}">
          <hardwareInterface>PositionJointInterface</hardwareInterface>
       </joint>
