Commit message: updated gripper

File: ezgripper_description/urdf/ezgripper_triple_mount.urdf.xacro (robot description, xacro)
@@ -1,5 +1,5 @@
 <?xml version="1.0" encoding="UTF-8"?>
 <robot name="ezgripper" xmlns:xacro="http://ros.org/wiki/xacro">
-<!--macro name="ezgripper_triple_mount" params="*origin"-->
+<xacro:include filename="$(find minilift_description)/urdf/macros.xacro" />
 <xacro:macro name="ezgripper_triple_mount" params="prefix parent_link *origin">
 <!-- links -->
@@ -10,4 +10,5 @@
           <mesh filename="package://ezgripper_description/meshes/visual/SAKE_Triple_Mount.stl"/>
         </geometry>
+        <material name="dark_grey"/>
       </visual>
       <collision>
@@ -22,4 +23,7 @@
     </inertial>
     </link>
+    <gazebo reference="${prefix}_ezgripper_mount">
+      <material>Gazebo/DarkGrey</material>
+    </gazebo>
     <joint name="${prefix}_ezgripper_mount2base" type="fixed">
         <origin rpy="0 0 0" xyz="0.0 0.0 0.0"/>
@@ -46,4 +50,5 @@
           <mesh filename="package://ezgripper_description/meshes/visual/SAKE_Palm_IM.stl"/>
         </geometry>
+        <material name="dark_grey"/>
       </visual>
       <collision>
@@ -58,4 +63,7 @@
     </inertial>
     </link>
+    <gazebo reference="${prefix}_ezgripper_palm_link">
+      <material>Gazebo/DarkGrey</material>
+    </gazebo>
     <joint name="${prefix}_ezgripper_mount2palm" type="fixed">
         <xacro:insert_block name="origin"/>
@@ -88,4 +96,5 @@
           <mesh filename="package://ezgripper_description/meshes/visual/SAKE_Finger_L1_IM.stl"/>
         </geometry>
+        <material name="dark_grey"/>
       </visual>
       <collision>
@@ -100,4 +109,7 @@
       </inertial>
     </link>
+    <gazebo reference="${prefix}_ezgripper_finger_L1_${postfix}">
+      <material>Gazebo/DarkGrey</material>
+    </gazebo>
 </xacro:macro>
 <xacro:macro name="ezgripper_finger_L2" params="prefix postfix reflect">
@@ -108,4 +120,5 @@
           <mesh filename="package://ezgripper_description/meshes/visual/SAKE_Finger_L2_IM.stl"/>
         </geometry>
+        <material name="dark_grey"/>
       </visual>
       <collision>
@@ -120,4 +133,7 @@
       </inertial>
     </link>
+    <gazebo reference="${prefix}_ezgripper_finger_L2_${postfix}">
+      <material>Gazebo/DarkGrey</material>
+    </gazebo>
 </xacro:macro>
 <xacro:macro name="ezgripper_finger_pad" params="prefix postfix reflect">
@@ -128,4 +144,5 @@
           <mesh filename="package://ezgripper_description/meshes/visual/SAKE_Finger_Pad_IM.stl"/>
         </geometry>
+        <material name="dark_grey"/>
       </visual>
       <collision>
@@ -140,4 +157,7 @@
       </inertial>
     </link>
+    <gazebo reference="${prefix}_ezgripper_finger_pad_${postfix}">
+      <material>Gazebo/DarkGrey</material>
+    </gazebo>
 </xacro:macro>
     <!-- joints -->
@@ -160,5 +180,5 @@
       <origin xyz="0.0595 ${reflectY*0.03} 0" rpy="${1.5708 * reflectR} 0 0"/>
       <axis xyz="0 1 0"/>
-      <limit lower=".27" upper="-1.57075" effort="1" velocity="3.67"/>
+      <limit lower="-1.57075" upper=".27" effort="1" velocity="3.67"/>
       <xacro:if value="${mimic_test}">
            <mimic joint="${prefix}_ezgripper_knuckle_palm_L1_1"/>

Commit message: removed redundant publishers

File: ezgripper_description/urdf/ezgripper_triple_mount.urdf.xacro (robot description, xacro)
@@ -223,13 +223,13 @@
 </xacro:macro>
 <xacro:macro name="gazebo_knuckle_jsp" params="prefix">
-   <gazebo>
+   <!-- <gazebo>
      <plugin name="joint_state_publisher" filename="libgazebo_ros_joint_state_publisher.so">
        <jointName>${prefix}_ezgripper_knuckle_palm_L1_1,${prefix}_ezgripper_knuckle_palm_L1_2  </jointName>
      </plugin>
-   </gazebo>
-</xacro:macro>
-<gazebo>
+   </gazebo> -->
+</xacro:macro>
+<!-- <gazebo>
    <plugin name="gazebo_ros_control" filename="libgazebo_ros_control.so">
    </plugin>
-</gazebo>
+</gazebo> -->
 </robot>

Commit message: added control parameter

File: ezgripper_description/urdf/ezgripper_triple_mount.urdf.xacro (robot description, xacro)
@@ -1,4 +1,6 @@
 <?xml version="1.0" encoding="UTF-8"?>
 <robot name="ezgripper" xmlns:xacro="http://ros.org/wiki/xacro">
+<!-- Toggle old behaviour -->
+<xacro:arg name="activate_control" default="false" />
 <xacro:include filename="$(find minilift_description)/urdf/macros.xacro" />
 <xacro:macro name="ezgripper_triple_mount" params="prefix parent_link *origin">
@@ -223,13 +225,17 @@
 </xacro:macro>
 <xacro:macro name="gazebo_knuckle_jsp" params="prefix">
-   <!-- <gazebo>
-     <plugin name="joint_state_publisher" filename="libgazebo_ros_joint_state_publisher.so">
-       <jointName>${prefix}_ezgripper_knuckle_palm_L1_1,${prefix}_ezgripper_knuckle_palm_L1_2  </jointName>
-     </plugin>
-   </gazebo> -->
-</xacro:macro>
-<!-- <gazebo>
-   <plugin name="gazebo_ros_control" filename="libgazebo_ros_control.so">
-   </plugin>
-</gazebo> -->
+  <xacro:if value="$(arg activate_control)">
+    <gazebo>
+      <plugin name="joint_state_publisher" filename="libgazebo_ros_joint_state_publisher.so">
+        <jointName>${prefix}_ezgripper_knuckle_palm_L1_1,${prefix}_ezgripper_knuckle_palm_L1_2  </jointName>
+      </plugin>
+    </gazebo>
+  </xacro:if>
+</xacro:macro>
+<xacro:if value="$(arg activate_control)">
+  <gazebo>
+    <plugin name="gazebo_ros_control" filename="libgazebo_ros_control.so">
+    </plugin>
+ </gazebo>
+</xacro:if>
 </robot>

Commit message: Updated Serial Dependency and moved control plugin

File: ezgripper_description/urdf/ezgripper_triple_mount.urdf.xacro (robot description, xacro)
@@ -1,6 +1,4 @@
 <?xml version="1.0" encoding="UTF-8"?>
 <robot name="ezgripper" xmlns:xacro="http://ros.org/wiki/xacro">
-<!-- Toggle old behaviour -->
-<xacro:arg name="activate_control" default="false" />
 <xacro:include filename="$(find minilift_description)/urdf/macros.xacro" />
 <xacro:macro name="ezgripper_triple_mount" params="prefix parent_link *origin">
@@ -35,13 +33,13 @@
         <limit effort="0" lower="-1.57075" upper="0.25" velocity="3.67"/>
     </joint>
-    <ezgripper_palm prefix="${prefix}1" parent_link="${prefix}_ezgripper_mount">
-    <origin xyz = "0.01 0.0 0.068" rpy = "0 0 0"/>
-    </ezgripper_palm>
-    <ezgripper_palm prefix="${prefix}2" parent_link="${prefix}_ezgripper_mount">
-    <origin xyz = "0.01 0.0 0" rpy = "0 0 0"/>
-    </ezgripper_palm>
-    <ezgripper_palm prefix="${prefix}3" parent_link="${prefix}_ezgripper_mount">
-    <origin xyz = "0.01 0.0 -0.068" rpy = "0 0 0"/>
-    </ezgripper_palm>
+    <xacro:ezgripper_palm prefix="${prefix}1" parent_link="${prefix}_ezgripper_mount">
+      <origin xyz = "0.01 0.0 0.068" rpy = "0 0 0"/>
+    </xacro:ezgripper_palm>
+    <xacro:ezgripper_palm prefix="${prefix}2" parent_link="${prefix}_ezgripper_mount">
+      <origin xyz = "0.01 0.0 0" rpy = "0 0 0"/>
+    </xacro:ezgripper_palm>
+    <xacro:ezgripper_palm prefix="${prefix}3" parent_link="${prefix}_ezgripper_mount">
+      <origin xyz = "0.01 0.0 -0.068" rpy = "0 0 0"/>
+    </xacro:ezgripper_palm>
 </xacro:macro>
 <xacro:macro name="ezgripper_palm" params="prefix parent_link *origin">
@@ -75,19 +73,19 @@
         <limit effort="0" lower="-1.57075" upper="0.25" velocity="3.67"/>
     </joint>
-    <ezgripper_finger_L1 prefix="${prefix}" postfix="1" reflect="1" />
-    <ezgripper_finger_L1 prefix="${prefix}" postfix="2" reflect="1" />
-    <ezgripper_finger_L2 prefix="${prefix}" postfix="1" reflect="1" />
-    <ezgripper_finger_L2 prefix="${prefix}" postfix="2" reflect="1" />
-    <ezgripper_finger_pad prefix="${prefix}" postfix="1" reflect="1" />
-    <ezgripper_finger_pad prefix="${prefix}" postfix="2" reflect="1" />
-    <ezgripper_knuckle_palm_L1 prefix="${prefix}" postfix="1" reflectY="1" reflectZ="1" reflectR="-1" mimic_test="false"/>
-    <ezgripper_knuckle_palm_L1 prefix="${prefix}" postfix="2" reflectY="-1" reflectZ="1" reflectR="1" mimic_test="false"/>
-    <ezgripper_knuckle_L1_L2 prefix="${prefix}" postfix="1" reflectY="1" reflectZ="1" reflectR="-1" mimic_test="false"/>
-    <ezgripper_knuckle_L1_L2 prefix="${prefix}" postfix="2" reflectY="-1" reflectZ="1" reflectR="1" mimic_test="false"/>
-    <ezgripper_joint_finger_pad prefix="${prefix}" postfix="1" reflectY="1" reflectZ="1" reflectR="1" mimic_test="false"/>
-    <ezgripper_joint_finger_pad prefix="${prefix}" postfix="2" reflectY="-1" reflectZ="1" reflectR="-1" mimic_test="false"/>
-    <ezgripper_knuckle_trans prefix="${prefix}" postfix="1"/>
-    <ezgripper_knuckle_trans prefix="${prefix}" postfix="2"/>
-    <gazebo_knuckle_jsp prefix="${prefix}" />
+    <xacro:ezgripper_finger_L1 prefix="${prefix}" postfix="1" reflect="1" />
+    <xacro:ezgripper_finger_L1 prefix="${prefix}" postfix="2" reflect="1" />
+    <xacro:ezgripper_finger_L2 prefix="${prefix}" postfix="1" reflect="1" />
+    <xacro:ezgripper_finger_L2 prefix="${prefix}" postfix="2" reflect="1" />
+    <xacro:ezgripper_finger_pad prefix="${prefix}" postfix="1" reflect="1" />
+    <xacro:ezgripper_finger_pad prefix="${prefix}" postfix="2" reflect="1" />
+    <xacro:ezgripper_knuckle_palm_L1 prefix="${prefix}" postfix="1" reflectY="1" reflectZ="1" reflectR="-1" mimic_test="false"/>
+    <xacro:ezgripper_knuckle_palm_L1 prefix="${prefix}" postfix="2" reflectY="-1" reflectZ="1" reflectR="1" mimic_test="false"/>
+    <xacro:ezgripper_knuckle_L1_L2 prefix="${prefix}" postfix="1" reflectY="1" reflectZ="1" reflectR="-1" mimic_test="false"/>
+    <xacro:ezgripper_knuckle_L1_L2 prefix="${prefix}" postfix="2" reflectY="-1" reflectZ="1" reflectR="1" mimic_test="false"/>
+    <xacro:ezgripper_joint_finger_pad prefix="${prefix}" postfix="1" reflectY="1" reflectZ="1" reflectR="1" mimic_test="false"/>
+    <xacro:ezgripper_joint_finger_pad prefix="${prefix}" postfix="2" reflectY="-1" reflectZ="1" reflectR="-1" mimic_test="false"/>
+    <xacro:ezgripper_knuckle_trans prefix="${prefix}" postfix="1"/>
+    <xacro:ezgripper_knuckle_trans prefix="${prefix}" postfix="2"/>
+    <xacro:gazebo_knuckle_jsp prefix="${prefix}" />
 </xacro:macro>
 <xacro:macro name="ezgripper_finger_L1" params="prefix postfix reflect">
@@ -225,17 +223,14 @@
 </xacro:macro>
 <xacro:macro name="gazebo_knuckle_jsp" params="prefix">
-  <xacro:if value="$(arg activate_control)">
-    <gazebo>
-      <plugin name="joint_state_publisher" filename="libgazebo_ros_joint_state_publisher.so">
-        <jointName>${prefix}_ezgripper_knuckle_palm_L1_1,${prefix}_ezgripper_knuckle_palm_L1_2  </jointName>
-      </plugin>
-    </gazebo>
-  </xacro:if>
-</xacro:macro>
-<xacro:if value="$(arg activate_control)">
   <gazebo>
-    <plugin name="gazebo_ros_control" filename="libgazebo_ros_control.so">
+    <plugin name="joint_state_publisher" filename="libgazebo_ros_joint_state_publisher.so">
+      <jointName>${prefix}_ezgripper_knuckle_palm_L1_1,${prefix}_ezgripper_knuckle_palm_L1_2  </jointName>
     </plugin>
- </gazebo>
-</xacro:if>
+  </gazebo>
+</xacro:macro>
+<gazebo>
+  <plugin name="gazebo_ros_control" filename="libgazebo_ros_control.so">
+    <robotNamespace>/minilift</robotNamespace>
+  </plugin>
+</gazebo>
 </robot>

Commit message: Reverted control parameter for octomap issues

File: ezgripper_description/urdf/ezgripper_triple_mount.urdf.xacro (robot description, xacro)
@@ -1,4 +1,6 @@
 <?xml version="1.0" encoding="UTF-8"?>
 <robot name="ezgripper" xmlns:xacro="http://ros.org/wiki/xacro">
+<!-- Toggle old behaviour -->
+<xacro:arg name="activate_control" default="false" />
 <xacro:include filename="$(find minilift_description)/urdf/macros.xacro" />
 <xacro:macro name="ezgripper_triple_mount" params="prefix parent_link *origin">
@@ -223,14 +225,17 @@
 </xacro:macro>
 <xacro:macro name="gazebo_knuckle_jsp" params="prefix">
+  <xacro:if value="$(arg activate_control)">
+    <gazebo>
+      <plugin name="joint_state_publisher" filename="libgazebo_ros_joint_state_publisher.so">
+        <jointName>${prefix}_ezgripper_knuckle_palm_L1_1,${prefix}_ezgripper_knuckle_palm_L1_2  </jointName>
+      </plugin>
+    </gazebo>
+  </xacro:if>
+</xacro:macro>
+<xacro:if value="$(arg activate_control)">
   <gazebo>
-    <plugin name="joint_state_publisher" filename="libgazebo_ros_joint_state_publisher.so">
-      <jointName>${prefix}_ezgripper_knuckle_palm_L1_1,${prefix}_ezgripper_knuckle_palm_L1_2  </jointName>
+    <plugin name="gazebo_ros_control" filename="libgazebo_ros_control.so">
     </plugin>
-  </gazebo>
-</xacro:macro>
-<gazebo>
-  <plugin name="gazebo_ros_control" filename="libgazebo_ros_control.so">
-    <robotNamespace>/minilift</robotNamespace>
-  </plugin>
-</gazebo>
+ </gazebo>
+</xacro:if>
 </robot>
